File: qfn/qfn-Badge.kicad_pcb (KiCad board)
At the start: 2 copper layers, 50 x 50 mm, 1 part

Commit message: JLC adjustments
Other:
- board text added: "Made in Shenzhen, China"
- board text removed: "In Shenzhen, China"
Changed lines of the file:
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@@
 		(stroke
 			(width 0.2)
-			(type default)
+			(type solid)
 		)
-		(fill no)
+		(fill yes)
 		(layer "Edge.Cuts")
 	)
-	(gr_text "In Shenzhen,\nChina"
-		(at 129 96 -0)
+	(gr_text "Made in \nShenzhen, China"
+		(at 127 90 0)
 		(layer "B.Cu")
 		(effects
 			(font
-				(size 3 3)
-				(bold yes)
+				(size 2 2)
 			)
 			(justify left bottom mirror)
